Commit message: fix some bags v1

File: tsukuba2023/urdf/orange.xacro (robot description, xacro)
@@ -16,27 +16,27 @@
   </xacro:macro>
   <!-- Import gazebo reference -->
-  <xacro:include filename="$(find igvc2023)/urdf/orange.gazebo"/>
+  <xacro:include filename="$(find tsukuba2023)/urdf/orange.gazebo"/>
   <!-- Import 2D LiDAR model -->
-  <xacro:include filename="$(find igvc2023)/urdf/sensors/hokuyo.urdf.xacro"/>
+  <xacro:include filename="$(find tsukuba2023)/urdf/sensors/hokuyo.urdf.xacro"/>
   <xacro:sensor_hokuyo name="hokuyo" parent="base_link" min_angle="-1.22" max_angle="1.22" samples="720">
     <origin xyz="0.16 0.0 0.05" rpy="0.0 0.0 0.0"/>
   </xacro:sensor_hokuyo>
   <!-- Import 3D LiDAR model -->
-  <xacro:include filename="$(find igvc2023)/urdf/sensors/velodyne.urdf.xacro"/>
+  <xacro:include filename="$(find tsukuba2023)/urdf/sensors/velodyne.urdf.xacro"/>
   <xacro:sensor_velodyne name="velodyne" parent="base_link" min_angle="-2.35619" max_angle="2.35619" samples="720">
     <origin xyz="-0.13 0.0 0.70" rpy="0.0 0.0 0.0"/>
   </xacro:sensor_velodyne>
   <!-- Import imu model -->
-  <xacro:include filename="$(find igvc2023)/urdf/sensors/imu.urdf.xacro"/>
+  <xacro:include filename="$(find tsukuba2023)/urdf/sensors/imu.urdf.xacro"/>
   <xacro:sensor_imu name="imu" parent="base_link" size="0.05 0.05 0.05">
     <origin xyz="0 0.0 0.068" rpy="0.0 0.0 0.0"/>
   </xacro:sensor_imu>
   <!-- Import fisheye camera model -->
-  <xacro:include filename="$(find igvc2023)/urdf/sensors/camera.urdf.xacro"/>
+  <xacro:include filename="$(find tsukuba2023)/urdf/sensors/camera.urdf.xacro"/>
   <xacro:sensor_camera name="camera" parent="base_link">
     <origin xyz="-0.13 0 1" rpy="0 0 0"/>
   </xacro:sensor_camera>
   <!-- Import gps model -->
-  <xacro:include filename="$(find igvc2023)/urdf/sensors/gps.urdf.xacro"/>
+  <xacro:include filename="$(find tsukuba2023)/urdf/sensors/gps.urdf.xacro"/>
   <xacro:sensor_gps name="gps" parent="base_link">
     <origin xyz="0.5 0 0.75" rpy="0 ${PI} 0"/>
@@ -60,5 +60,5 @@
       <origin xyz="-0.355 0.0 0.3" rpy="0.0 0.0 0.0"/>
       <geometry>
-        <mesh filename="package://igvc2023/meshes/IGVCchassis.dae"/>
+        <mesh filename="package://tsukuba2023/meshes/IGVCchassis.dae"/>
       </geometry>
     </visual>
@@ -90,5 +90,5 @@
       <origin xyz="-0.735 0.10 -0.039" rpy="0.0 0.0 0.0"/>
       <geometry>
-        <mesh filename="package://igvc2023/meshes/left_back_wheel.dae"/>
+        <mesh filename="package://tsukuba2023/meshes/left_back_wheel.dae"/>
       </geometry>
     </visual>
@@ -104,5 +104,5 @@
       <origin xyz="-0.735 -0.10 -0.039" rpy="0.0 0.0 0.0"/>
       <geometry>
-        <mesh filename="package://igvc2023/meshes/right_back_wheel.dae"/>
+        <mesh filename="package://tsukuba2023/meshes/right_back_wheel.dae"/>
         <sphere radius="0.0625"/>
       </geometry>
@@ -134,5 +134,5 @@
       <origin xyz="0.0 0.0 0.0" rpy="0.0 0.0 0.0"/>
       <geometry>
-        <mesh filename="package://igvc2023/meshes/front_wheel.dae"/>
+        <mesh filename="package://tsukuba2023/meshes/front_wheel.dae"/>
       </geometry>
     </visual>
@@ -153,5 +153,5 @@
       <origin xyz="0.0 0.0 0.0" rpy="0.0 0.0 0.0"/>
       <geometry>
-        <mesh filename="package://igvc2023/meshes/front_wheel.dae"/>
+        <mesh filename="package://tsukuba2023/meshes/front_wheel.dae"/>
       </geometry>
     </visual>

File: tsukuba2023/urdf/sensors/hokuyo.urdf.xacro (robot description, xacro)
@@ -21,5 +21,5 @@
         <origin xyz="0 0 0" rpy="0 0 0"/>
         <geometry>
-          <mesh filename="package://igvc2023/meshes/hokuyo.dae"/>
+          <mesh filename="package://tsukuba2023/meshes/hokuyo.dae"/>
         </geometry>
       </visual>

File: tsukuba2023/urdf/sensors/velodyne.urdf.xacro (robot description, xacro)
@@ -21,5 +21,5 @@
         <origin xyz="0 0 0" rpy="0 0 0"/>
         <geometry>
-          <mesh filename="package://igvc2023/meshes/velodyne.dae"/>
+          <mesh filename="package://tsukuba2023/meshes/velodyne.dae"/>
         </geometry>
       </visual>

Commit message: fix some bags v5

File: tsukuba2023/urdf/orange.xacro (robot description, xacro)
@@ -20,10 +20,10 @@
   <xacro:include filename="$(find tsukuba2023)/urdf/sensors/hokuyo.urdf.xacro"/>
   <xacro:sensor_hokuyo name="hokuyo" parent="base_link" min_angle="-1.22" max_angle="1.22" samples="720">
-    <origin xyz="0.16 0.0 0.05" rpy="0.0 0.0 0.0"/>
+    <origin xyz="0.16 0.0 0.1" rpy="0.0 0.0 0.0"/>
   </xacro:sensor_hokuyo>
   <!-- Import 3D LiDAR model -->
   <xacro:include filename="$(find tsukuba2023)/urdf/sensors/velodyne.urdf.xacro"/>
   <xacro:sensor_velodyne name="velodyne" parent="base_link" min_angle="-2.35619" max_angle="2.35619" samples="720">
-    <origin xyz="-0.13 0.0 0.70" rpy="0.0 0.0 0.0"/>
+    <origin xyz="-0.10 0.0 0.95" rpy="0.0 0.0 0.0"/>
   </xacro:sensor_velodyne>
   <!-- Import imu model -->
@@ -32,13 +32,13 @@
     <origin xyz="0 0.0 0.068" rpy="0.0 0.0 0.0"/>
   </xacro:sensor_imu>
-  <!-- Import fisheye camera model -->
+  <!-- Import fisheye camera model >
   <xacro:include filename="$(find tsukuba2023)/urdf/sensors/camera.urdf.xacro"/>
   <xacro:sensor_camera name="camera" parent="base_link">
     <origin xyz="-0.13 0 1" rpy="0 0 0"/>
-  </xacro:sensor_camera>
+  </xacro:sensor_camera-->
   <!-- Import gps model -->
   <xacro:include filename="$(find tsukuba2023)/urdf/sensors/gps.urdf.xacro"/>
   <xacro:sensor_gps name="gps" parent="base_link">
-    <origin xyz="0.5 0 0.75" rpy="0 ${PI} 0"/>
+    <origin xyz="0.6 0 0.65" rpy="0 ${PI} 0"/>
   </xacro:sensor_gps>
   <!-- Base Footprint -->
@@ -52,19 +52,19 @@
   <link name="base_link">
     <collision>
-      <origin xyz="-0.33 0.0 0.25" rpy="0.0 0.0 0.0"/>
+      <origin xyz="-0.07 0.0 0.55" rpy="0.0 0.0 0.0"/>
       <geometry>
-        <box size="0.9 0.5 0.5"/>
+        <box size="0.7 0.5 1"/>
       </geometry>
     </collision>
     <visual>
-      <origin xyz="-0.355 0.0 0.3" rpy="0.0 0.0 0.0"/>
+      <origin xyz="0 0.0 0" rpy="0.0 0.0 0.0"/>
       <geometry>
-        <mesh filename="package://tsukuba2023/meshes/IGVCchassis.dae"/>
+        <mesh filename="package://tsukuba2023/meshes/Chassis.dae"/>
       </geometry>
     </visual>
     <inertial>
        <mass value="40" />
-       <origin xyz="-0.33 0.0 0.26" rpy="0.0 0.0 0.0"/>
-       <xacro:box_inertia m="40" x="0.9" y="0.5" z="0.45"/>
+       <origin xyz="-0.07 0.0 0.55" rpy="0.0 0.0 0.0"/>
+       <xacro:box_inertia m="40" x="0.67" y="0.5" z="1."/>
     </inertial>
   </link>
@@ -80,7 +80,13 @@
     <parent link="base_link"/>
   </joint>
+  <!-- Forward wheels -->
+  <joint name="forward_caster_hinge" type ="fixed">
+    <origin xyz="0.0 0.0 0.0" rpy="0.0 0.0 0.0"/>
+    <child link="forward_caster_link"/>
+    <parent link="base_link"/>
+  </joint>
   <link name="left_caster_link">
     <collision>
-      <origin xyz="-0.735 0.10 -0.039" rpy="0.0 ${PI/2} ${PI/2}"/>
+      <origin xyz="-0.35 0.10 -0.039" rpy="0.0 ${PI/2} ${PI/2}"/>
       <geometry>
         <sphere radius="0.0625"/>
@@ -88,5 +94,5 @@
     </collision>
     <visual>
-      <origin xyz="-0.735 0.10 -0.039" rpy="0.0 0.0 0.0"/>
+      <origin xyz="-0.35 0.10 -0.039" rpy="0.0 0.0 0.0"/>
       <geometry>
         <mesh filename="package://tsukuba2023/meshes/left_back_wheel.dae"/>
@@ -96,5 +102,5 @@
   <link name="right_caster_link">
     <collision>
-      <origin xyz="-0.735 -0.10 -0.039" rpy="0.0 ${PI/2} ${PI/2}"/>
+      <origin xyz="-0.35 -0.10 -0.039" rpy="0.0 ${PI/2} ${PI/2}"/>
       <geometry>
         <sphere radius="0.0625"/>
@@ -102,5 +108,20 @@
     </collision>
     <visual>
-      <origin xyz="-0.735 -0.10 -0.039" rpy="0.0 0.0 0.0"/>
+      <origin xyz="-0.35 -0.10 -0.039" rpy="0.0 0.0 0.0"/>
+      <geometry>
+        <mesh filename="package://tsukuba2023/meshes/right_back_wheel.dae"/>
+        <sphere radius="0.0625"/>
+      </geometry>
+    </visual>
+  </link>
+  <link name="forward_caster_link">
+    <collision>
+      <origin xyz="0.2 0 -0.039" rpy="0.0 ${PI/2} ${PI/2}"/>
+      <geometry>
+        <sphere radius="0.0625"/>
+      </geometry>
+    </collision>
+    <visual>
+      <origin xyz="0.2 0 -0.039" rpy="0.0 0.0 0.0"/>
       <geometry>
         <mesh filename="package://tsukuba2023/meshes/right_back_wheel.dae"/>

Commit message: fix position of hokuyo and add nakaniwa.stl

File: tsukuba2023/urdf/orange.xacro (robot description, xacro)
@@ -20,5 +20,5 @@
   <xacro:include filename="$(find tsukuba2023)/urdf/sensors/hokuyo.urdf.xacro"/>
   <xacro:sensor_hokuyo name="hokuyo" parent="base_link" min_angle="-1.22" max_angle="1.22" samples="720">
-    <origin xyz="0.16 0.0 0.1" rpy="0.0 0.0 0.0"/>
+    <origin xyz="0.25 0.0 0.1" rpy="0.0 0.0 0.0"/>
   </xacro:sensor_hokuyo>
   <!-- Import 3D LiDAR model -->

File: tsukuba2023/urdf/sensors/hokuyo.urdf.xacro (robot description, xacro)
@@ -45,5 +45,5 @@
         </scan>
         <range>
-          <min>0.10</min>
+          <min>0.20</min>
           <max>30.0</max>
           <resolution>0.01</resolution>
